Commit message: IK final

File: urdf/finale1.urdf (robot description, URDF)
Before this commit: robot finale, 7 links, 6 joints
Joints:
- joint j2: limit lower=-3.14 upper=3.14 effort=100 velocity=0.1 -> lower=-3.78 upper=0.64 effort=100 velocity=0.1
- joint j3: limit lower=-3.14 upper=3.14 effort=100 velocity=0.1 -> lower=-2.8 upper=2.8 effort=100 velocity=0.1
- joint j4: limit lower=-3.14 upper=3.14 effort=100 velocity=0.1 -> lower=-2 upper=2 effort=100 velocity=0.1
